File: pwmcontroller.sch (KiCad schematic (older format))
At the start: 13 parts, among them J1 CONN_01X04, J2 CONN_01X04, U1 WPMIx9200501S, U2 NE555

Commit message: Fix component values
Parts:
- R1: value 100K -> 1K
Changed lines of the file:
@@
 P 4650 3500
 F 0 "R1" V 4730 3500 50  0000 C CNN
-F 1 "100K" V 4650 3500 50  0000 C CNN
+F 1 "1K" V 4650 3500 50  0000 C CNN
 F 2 "Resistors_THT:R_Axial_DIN0207_L6.3mm_D2.5mm_P10.16mm_Horizontal" V 4580 3500 50  0001 C CNN
 F 3 "" H 4650 3500 50  0001 C CNN
