File: pwmcontroller.kicad_pcb (KiCad board)
At the start: 2 copper layers, 35.1 x 44.5 mm, 19 parts, among them J1 CONN_01X04, J2 CONN_01X04, U1 WPMIx9200501S, U2 NE555

Commit message: Change C2 to 470pF
After doing some breadboard testing the carrier frequency of the PWM
signal was too low at only ~12kHz to ~14kHz. The PWM fan spec says this
needs to be nominally 25kHz with a range of 21kHz to 28kHz. By
decreasing the capacitance of the C2 to 470pF from 680pF this should
adjust the frequency to be in this range. Next time I'll do the
arithmetic before ordering parts.
Parts:
- C2: value 680pF -> 470pF
Changed lines of the file:
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@@
     (links 26)
     (no_connects 0)
-    (area 139.370999 88.513 174.765001 135.869)
+    (area 139.370999 89.840999 174.573001 134.441001)
     (thickness 1.6)
     (drawings 7)
@@
   (layers
     (0 F.Cu signal)
-    (31 B.Cu signal hide)
+    (31 B.Cu signal)
     (32 B.Adhes user hide)
     (33 F.Adhes user)
@@
       (effects (font (size 1 1) (thickness 0.15)))
     )
-    (fp_text value 680pF (at 2.5 2.56 90) (layer F.Fab)
-      (effects (font (size 1 1) (thickness 0.15)))
-    )
+    (fp_text value 470pF (at 2.5 2.56 90) (layer F.Fab)
+      (effects (font (size 1 1) (thickness 0.15)))
+    )
